Commit message: Running Project

File: ros2_ws/src/vrc_system/urdf/advanced_humanoid_robot.urdf (robot description, URDF)
Before this commit: robot advanced_humanoid_robot, 25 links, 24 joints
Links:
- removed link left_arm
- removed link left_foot
- removed link left_shin
- removed link left_thigh
- removed link right_arm
- removed link right_foot
- removed link right_shin
- removed link right_thigh
- added link head_visor, mass 0.1; collision box size=0.03 0.14 0.05; visual box size=0.03 0.14 0.05
- added link left_eye, mass 0.02; collision sphere radius=0.025; visual sphere radius=0.025
- added link left_eyebrow; visual box size=0.05 0.01 0.01
- added link left_finger1, mass 0.02; collision box size=0.04 0.012 0.012; visual box size=0.04 0.012 0.012
- added link left_finger2, mass 0.02; collision box size=0.04 0.012 0.012; visual box size=0.04 0.012 0.012
- added link left_forearm, mass 0.25; collision cylinder length=0.12 radius=0.02; visual cylinder length=0.12 radius=0.02
- added link left_palm, mass 0.1; collision box size=0.08 0.04 0.02; visual box size=0.08 0.04 0.02
- added link left_upper_arm, mass 0.3; collision cylinder length=0.12 radius=0.022; visual cylinder length=0.12 radius=0.022
- added link left_wrist, mass 0.08; collision sphere radius=0.03; visual sphere radius=0.03
- added link mouth, mass 0.02; collision box size=0.06 0.015 0.012; visual box size=0.06 0.015 0.012
- added link nose, mass 0.01; collision box size=0.02 0.02 0.02; visual box size=0.02 0.02 0.02
- added link right_eye, mass 0.02; collision sphere radius=0.025; visual sphere radius=0.025
- added link right_eyebrow; visual box size=0.05 0.01 0.01
- added link right_finger1, mass 0.02; collision box size=0.04 0.012 0.012; visual box size=0.04 0.012 0.012
- added link right_finger2, mass 0.02; collision box size=0.04 0.012 0.012; visual box size=0.04 0.012 0.012
- added link right_forearm, mass 0.25; collision cylinder length=0.12 radius=0.02; visual cylinder length=0.12 radius=0.02
- added link right_palm, mass 0.1; collision box size=0.08 0.04 0.02; visual box size=0.08 0.04 0.02
- added link right_upper_arm, mass 0.3; collision cylinder length=0.12 radius=0.022; visual cylinder length=0.12 radius=0.022
- added link right_wrist, mass 0.08; collision sphere radius=0.03; visual sphere radius=0.03
- link base_link: mass 5.0 -> 10.0
- link chest_panel: mass None -> 0.3; geometry collision box size=0.02 0.12 0.14; visual box size=0.02 0.12 0.14
- link head: mass None -> 1.0; geometry collision sphere radius=0.11; visual sphere radius=0.11
- link head_top: mass None -> 0.1; geometry collision box size=0.13 0.13 0.02; visual box size=0.13 0.13 0.02
- link left_elbow_ring: mass None -> 0.08; geometry collision cylinder length=0.02 radius=0.028; visual cylinder length=0.02 radius=0.028
- link left_hip_pad: mass None -> 0.1; geometry collision box size=0.02 0.05 0.06; visual box size=0.02 0.05 0.06
- link left_shoulder: mass None -> 0.4; geometry collision sphere radius=0.055; visual sphere radius=0.055
- link left_shoulder_plate: mass None -> 0.2; geometry collision box size=0.10 0.06 0.02; visual box size=0.10 0.06 0.02
- link left_wheel: mass None -> 0.7; geometry collision cylinder length=0.035 radius=0.06; visual cylinder length=0.035 radius=0.06
- link pelvis: mass 3.0 -> 4.0
- link right_elbow_ring: mass None -> 0.08; geometry collision cylinder length=0.02 radius=0.028; visual cylinder length=0.02 radius=0.028
- link right_hip_pad: mass None -> 0.1; geometry collision box size=0.02 0.05 0.06; visual box size=0.02 0.05 0.06
- link right_shoulder: mass None -> 0.4; geometry collision sphere radius=0.055; visual sphere radius=0.055
- link right_shoulder_plate: mass None -> 0.2; geometry collision box size=0.10 0.06 0.02; visual box size=0.10 0.06 0.02
- link right_wheel: mass None -> 0.7; geometry collision cylinder length=0.035 radius=0.06; visual cylinder length=0.035 radius=0.06
- link torso: mass 4.0 -> 3.0
- link waist: mass None -> 2.0; geometry collision box size=0.18 0.13 0.06; visual box size=0.18 0.13 0.06
Joints:
- removed joint left_arm_joint
- removed joint left_elbow_ring_joint
- removed joint left_foot_joint
- removed joint left_shin_joint
- removed joint left_thigh_joint
- removed joint right_arm_joint
- removed joint right_elbow_ring_joint
- removed joint right_foot_joint
- removed joint right_shin_joint
- removed joint right_thigh_joint
- added joint head_visor_joint: type fixed, parent head, child head_visor
- added joint left_elbow_joint: type revolute, parent left_upper_arm, child left_elbow_ring, origin xyz=0 0 -0.12, axis 0 1 0, limit lower=0 upper=2.5 effort=5 velocity=2.0
- added joint left_eye_joint: type fixed, parent head, child left_eye
- added joint left_eyebrow_joint: type fixed, parent head, child left_eyebrow
- added joint left_finger1_joint: type revolute, parent left_palm, child left_finger1, origin xyz=0.04 0.02 0, axis 0 0 1, limit lower=0 upper=0.7 effort=1 velocity=2.0
- added joint left_finger2_joint: type revolute, parent left_palm, child left_finger2, origin xyz=0.04 -0.02 0, axis 0 0 -1, limit lower=0 upper=0.7 effort=1 velocity=2.0
- added joint left_forearm_joint: type fixed, parent left_elbow_ring, child left_forearm, origin xyz=0 0 0
- added joint left_palm_joint: type fixed, parent left_wrist, child left_palm, origin xyz=0 0 0
- added joint left_upper_arm_joint: type revolute, parent left_shoulder, child left_upper_arm, origin xyz=0 0 -0.04, axis 0 1 0, limit lower=-1.57 upper=1.57 effort=5 velocity=2.0
- added joint left_wrist_joint: type revolute, parent left_forearm, child left_wrist, origin xyz=0 0 -0.12, axis 0 0 1, limit lower=-1.2 upper=1.2 effort=2 velocity=2.0
- added joint mouth_joint: type fixed, parent head, child mouth
- added joint nose_joint: type fixed, parent head, child nose
- added joint right_elbow_joint: type revolute, parent right_upper_arm, child right_elbow_ring, origin xyz=0 0 -0.12, axis 0 1 0, limit lower=0 upper=2.5 effort=5 velocity=2.0
- added joint right_eye_joint: type fixed, parent head, child right_eye
- added joint right_eyebrow_joint: type fixed, parent head, child right_eyebrow
- added joint right_finger1_joint: type revolute, parent right_palm, child right_finger1, origin xyz=0.04 0.02 0, axis 0 0 1, limit lower=0 upper=0.7 effort=1 velocity=2.0
- added joint right_finger2_joint: type revolute, parent right_palm, child right_finger2, origin xyz=0.04 -0.02 0, axis 0 0 -1, limit lower=0 upper=0.7 effort=1 velocity=2.0
- added joint right_forearm_joint: type fixed, parent right_elbow_ring, child right_forearm, origin xyz=0 0 0
- added joint right_palm_joint: type fixed, parent right_wrist, child right_palm, origin xyz=0 0 0
- added joint right_upper_arm_joint: type revolute, parent right_shoulder, child right_upper_arm, origin xyz=0 0 -0.04, axis 0 1 0, limit lower=-1.57 upper=1.57 effort=5 velocity=2.0
- added joint right_wrist_joint: type revolute, parent right_forearm, child right_wrist, origin xyz=0 0 -0.12, axis 0 0 1, limit lower=-1.2 upper=1.2 effort=2 velocity=2.0
- joint head_joint: axis 0 0 1 -> (none); limit lower=-1.0 upper=1.0 effort=2 velocity=1.5 -> (none); origin xyz=0 0 0.20 -> xyz=0 0 0.22; type revolute -> fixed
- joint left_wheel_joint: origin xyz=0 0.11 -0.07 -> xyz=0 0.12 0; parent pelvis -> base_link
- joint right_wheel_joint: origin xyz=0 -0.11 -0.07 -> xyz=0 -0.12 0; parent pelvis -> base_link
